File: MartincitoClock/MartincitoClock copy.kicad_sch (KiCad schematic)
At the start: 22 parts, among them J2 PJ-102AH, SW1 Omron_B3F_SPST, U1 ATmega328-PU, U2 L7805, Y1 Crystal

Commit message: Week 2 Deliverable
Parts:
- removed C2, C7: C_0805_0.1uf, footprints:C_0805_2012Metric, symbol HPS:C_0805_0.1uf
- removed R3, R4: R_0805_47, footprints:R_0805_2012Metric, symbol HPS:R_0805_47
- removed SW1: Omron_B3F_SPST, footprints:SW_SPST_Omron_B3FS-100xP, symbol HPS:Omron_B3F_SPST
- removed U2: L7805, symbol HPS:L7805
- added C3, C4: C, footprints:C_0805_2012Metric, symbol HPS:C_0805_0.1uf
- added C5: CP, footprints:C_0805_2012Metric, symbol HPS:C_0805_0.1uf
- C1: value C_0805_1uf -> CP
- C2: value C_0805_0.1uf -> C
- renumbered J2 to J?
Connections:
- net GND: now also C3.1, C4.1, C5.1
- net VCC: now also C3.2, C4.2, C5.2
- net at R2.2, U1.1 (~{RESET}/PC6): now also C6.2
- net at U1.2 (PD0): now also J?.4 (Pin_4)
- net at U1.3 (PD1): now also J?.5 (Pin_5)
Other:
- note removed: "LED"
- note removed: "Power input"
- note removed: "Vf = 2v Vr = 3v 10mcd @ 1.35mA therefore R=2.2KOhm"
- moved on the sheet: C1, C6, J?, R2
