File: MartincitoClock/MartincitoClock.kicad_sch (KiCad schematic)
At the start: 49 parts, among them J1 Conn_01x06, J2 Power_inlet_vertical, J5 Conn_02x03_Odd_Even, SW1 Omron_B3F_SPST, SW2 Omron_B3F_SPST, SW3 Omron_B3F_SPST, U1 ATmega328-PU, U10 ADT7410, U2 L7805, U3 DS1307_DIP-8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

Commit message: Final Gerber
Parts:
- C1, C12: Voltage + -> N/A
- U2: Digikey PN (none) -> 497-7255-1-ND; MFG (none) -> STMicroelectronics; MPN (none) -> L7805CDT-TR
Connections:
- net RESET is gone; now on net Reset: J5.5 (Pin_5)
- no-connect marks 11 -> 12
Changed lines of the file:
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@@
   (no_connect (at 237.49 73.66))
   (no_connect (at 33.02 170.18))
+  (no_connect (at 67.31 133.35))
   (polyline (pts (xy 39.37 83.82) (xy 12.7 83.82))
     (stroke (width 0) (type default) (color 0 0 0 0))
@@
     )
   )
-  (global_label "RESET" (shape input) (at 148.59 25.4 0) (fields_autoplaced)
+  (global_label "Reset" (shape input) (at 148.59 25.4 0) (fields_autoplaced)
     (effects (font (size 1.27 1.27)) (justify left))
-    (property "Intersheet References" "${INTERSHEET_REFS}" (id 0) (at 156.7483 25.3206 0)
+    (property "Intersheet References" "${INTERSHEET_REFS}" (id 0) (at 156.2041 25.3206 0)
       (effects (font (size 1.27 1.27)) (justify left) hide)
     )
@@
     (pin "1")
   )
-  (symbol (lib_id "HPS:MountingHole") (at 39.37 185.42 0) (unit 1)
+  (symbol (lib_name "MountingHole_3") (lib_id "HPS:MountingHole") (at 39.37 185.42 0) (unit 1)
     (in_bom yes) (on_board yes) (fields_autoplaced)
     (property "Reference" "H3" (id 0) (at 41.91 184.1499 0)
@@
     (pin "2")
   )
-  (symbol (lib_id "HPS:MountingHole") (at 19.05 185.42 0) (unit 1)
+  (symbol (lib_name "MountingHole_1") (lib_id "HPS:MountingHole") (at 19.05 185.42 0) (unit 1)
     (in_bom yes) (on_board yes) (fields_autoplaced)
     (property "Reference" "H1" (id 0) (at 21.59 184.1499 0)
@@
       (effects (font (size 1.27 1.27)) hide)
     )
-    (property "Voltage" "+" (id 8) (at 50.8 170.1799 0)
+    (property "Voltage" "N/A" (id 8) (at 50.8 170.1799 0)
       (effects (font (size 1.27 1.27)) (justify right))
     )
@@
   (symbol (lib_id "HPS:DS1307_DIP-8") (at 54.61 133.35 0) (unit 1)
     (in_bom yes) (on_board yes)
-    (property "Reference" "U3" (id 0) (at 73.66 139.27 0))
-    (property "Value" "DS1307_DIP-8" (id 1) (at 73.66 141.27 0))
+    (property "Reference" "U3" (id 0) (at 63.5 137.16 0))
+    (property "Value" "DS1307_DIP-8" (id 1) (at 66.04 143.51 0))
     (property "Footprint" "footprints:DIP-8_W7.62mm" (id 2) (at 54.61 161.29 0)
       (effects (font (size 1.27 1.27)) hide)
@@
     (pin "1")
   )
-  (symbol (lib_id "HPS:MountingHole") (at 19.05 193.04 0) (unit 1)
+  (symbol (lib_name "MountingHole_2") (lib_id "HPS:MountingHole") (at 19.05 193.04 0) (unit 1)
     (in_bom yes) (on_board yes) (fields_autoplaced)
     (property "Reference" "H2" (id 0) (at 21.59 191.7699 0)
@@
       (effects (font (size 1.27 1.27)) hide)
     )
-    (property "Voltage" "+" (id 8) (at 96.52 165.1001 0)
+    (property "Voltage" "N/A" (id 8) (at 96.52 165.1001 0)
       (effects (font (size 1.27 1.27)) (justify left))
     )
@@
     (pin "1")
   )
-  (symbol (lib_name "L7805_1") (lib_id "HPS:L7805") (at 67.31 163.83 0) (unit 1)
+  (symbol (lib_id "HPS:L7805") (at 67.31 163.83 0) (unit 1)
     (in_bom yes) (on_board yes) (fields_autoplaced)
     (property "Reference" "U2" (id 0) (at 67.31 156.21 0))
@@
       (effects (font (size 1.27 1.27)) hide)
     )
+    (property "Digikey PN" "497-7255-1-ND" (id 4) (at 67.31 163.83 0)
+      (effects (font (size 1.27 1.27)) hide)
+    )
+    (property "MPN" "L7805CDT-TR" (id 5) (at 67.31 163.83 0)
+      (effects (font (size 1.27 1.27)) hide)
+    )
+    (property "MFG" "STMicroelectronics" (id 6) (at 67.31 163.83 0)
+      (effects (font (size 1.27 1.27)) hide)
+    )

Commit message: Revised Final
Parts:
- removed TP1, TP2, TP3, TP4: TestPoint, footprints:TestPoint_THTPad_D2.0mm_Drill1.0mm, symbol HPS:TestPoint
Connections:
- net D0: now also D2.5 (R8); no longer D2.13 (C1)
- net D1: now also D2.2 (R7); no longer D2.3 (C2)
- net D2: now also D2.7 (R6); no longer D2.4 (C3)
- net D3: now also D2.1 (R5); no longer D2.10 (C4)
- net D4: now also D2.12 (R4); no longer D2.6 (C5)
- net D5: now also D2.8 (R3); no longer D2.11 (C6)
- net D6: now also D2.14 (R2); no longer D2.15 (C7)
- net D7: now also D2.9 (R1); no longer D2.16 (C8)
- net DIN: now also U4.24 (DOUT), U6.1 (DIN); no longer U1.17 (MOSI/PB3), U4.1 (DIN)
- net DISP_CLK: now also U4.13 (CLK)
- net DISP_LOAD: now also U4.12 (LOAD)
- net LED_SCK: now also J5.3 (Pin_3)
- net MISO: now also U1.18 (MISO/PB4); no longer U1.4 (INT0/PD2)
- net MOSI: now also U1.17 (MOSI/PB3); no longer U1.11 (OC0B/PD5)
- net at U4.21 (SEG_E): now also D2.10 (C4); no longer D2.1 (R5)
- net at U4.23 (SEG_D): now also D2.6 (C5); no longer D2.12 (R4)
- net at U4.16 (SEG_B): now also D2.15 (C7); no longer D2.14 (R2)
- net at U4.17 (SEG_G): now also D2.3 (C2); no longer D2.2 (R7)
- net at U4.22 (SEG_DP): now also D2.13 (C1); no longer D2.5 (R8)
- net at U4.15 (SEG_F): now also D2.4 (C3); no longer D2.7 (R6)
- net at U4.20 (SEG_C): now also D2.11 (C6); no longer D2.8 (R3)
- net at U4.14 (SEG_A): now also D2.16 (C8); no longer D2.9 (R1)
- removed net CLK: U1.18 (MISO/PB4), U4.13 (CLK)
- net CS1: no longer names the net of U1.5 (INT1/PD3)
- net CS1: no longer U4.12 (LOAD)
- net DISP_DATA: no longer names the net of U1.16 (OC1B/PB2)
- net DISP_DATA: no longer U6.1 (DIN)
- net ISP: no longer names the net of U1.6 (PD4)
- net ISP: no longer J5.3 (Pin_3)
- new net DinMAX: U1.4 (INT0/PD2), U4.1 (DIN)
- no-connect marks 12 -> 15
Other:
- moved on the sheet: D2
