File: MartincitoClock/_autosave-MartincitoClock.kicad_pcb (KiCad board)
At the start: 2 copper layers, 140 x 90 mm, 49 parts, among them J1 Conn_01x06, J2 Power_inlet_vertical, J5 Conn_02x03_Odd_Even, SW1 Omron_B3F_SPST, SW2 Omron_B3F_SPST, SW3 Omron_B3F_SPST, U1 ATmega328-PU, U10 ADT7410, U2 L7805, U3 DS1307_DIP-8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

Commit message: Week 6
Week 6 Deliverable
Parts:
- D2: value KWM-30881CVB -> KWM-30881XVB
Connections:
- J5 pad 5: RESET -> Reset
Routing:
- net Reset: track 21.2 -> 32.9 mm, vias 0 -> 1
Other:
- board text added: "Ahora Yo Picheo"
