File: MartincitoClock/MartincitoClock.kicad_pcb (KiCad board)
At the start: 2 copper layers, 140 x 90 mm, 49 parts, among them J1 Conn_01x06, J2 Power_inlet_vertical, J5 Conn_02x03_Odd_Even, SW1 Omron_B3F_SPST, SW2 Omron_B3F_SPST, SW3 Omron_B3F_SPST, U1 ATmega328-PU, U10 ADT7410, U2 L7805, U3 DS1307_DIP-8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

Commit message: Final Gerber
Parts:
- added G***: LOGO, footprints:HPS_logo, F.Cu at (195.6, 116.8)
- D2: value KWM-30881CVB -> KWM-30881XVB
Connections:
- J5 pad 5: RESET -> Reset
Routing:
- net Reset: track 21.2 -> 32.9 mm, vias 0 -> 1
Other:
- board text added: "Ahora Yo Picheo"
- board text added: "HOUR"
- board text added: "MIN"
- board text added: "Martin Mejia Martinez"
- board text added: "SERIAL"

Commit message: Revised Final
Parts:
- removed TP1, TP2, TP3, TP4: TestPoint, footprints:TestPoint_THTPad_D2.0mm_Drill1.0mm
- D2: value KWM-30881XVB -> KWM-30881CVB
- moved G*** 2.54 mm to (198.1, 116.8)
Connections:
- D2 pad 1: Net-(D2-Pad1) -> D3
- D2 pad 10: D3 -> Net-(U4-Pad21)
- D2 pad 11: D5 -> Net-(D2-Pad11)
- D2 pad 12: Net-(D2-Pad12) -> D4
- D2 pad 13: D0 -> Net-(U4-Pad22)
- D2 pad 14: Net-(D2-Pad14) -> D6
- D2 pad 15: D6 -> Net-(U4-Pad16)
- D2 pad 16: D7 -> Net-(U4-Pad14)
- D2 pad 2: Net-(D2-Pad2) -> D1
- D2 pad 3: D1 -> Net-(U4-Pad17)
- D2 pad 4: D2 -> Net-(U4-Pad15)
- D2 pad 5: Net-(D2-Pad5) -> D0
- D2 pad 6: D4 -> Net-(U4-Pad23)
- D2 pad 7: Net-(D2-Pad7) -> D2
- D2 pad 8: Net-(D2-Pad8) -> D5
- D2 pad 9: Net-(D2-Pad9) -> D7
- J5 pad 3: ISP -> LED_SCK
- U1 pad 11: MOSI -> unconnected-(U1-Pad11)
- U1 pad 16: DISP_DATA -> unconnected-(U1-Pad16)
- U1 pad 17: DIN -> MOSI
- U1 pad 18: CLK -> MISO
- U1 pad 4: MISO -> DinMAX
- U1 pad 5: CS1 -> unconnected-(U1-Pad5)
- U1 pad 6: ISP -> unconnected-(U1-Pad6)
- U4 pad 1: DIN -> DinMAX
- U4 pad 12: CS1 -> DISP_LOAD
- U4 pad 13: CLK -> DISP_CLK
- U4 pad 14: Net-(D2-Pad9) -> Net-(U4-Pad14)
- U4 pad 15: Net-(D2-Pad7) -> Net-(U4-Pad15)
- U4 pad 16: Net-(D2-Pad14) -> Net-(U4-Pad16)
- U4 pad 17: Net-(D2-Pad2) -> Net-(U4-Pad17)
- U4 pad 20: Net-(D2-Pad8) -> Net-(D2-Pad11)
- U4 pad 21: Net-(D2-Pad1) -> Net-(U4-Pad21)
- U4 pad 22: Net-(D2-Pad5) -> Net-(U4-Pad22)
- U4 pad 23: Net-(D2-Pad12) -> Net-(U4-Pad23)
- U4 pad 24: unconnected-(U4-Pad24) -> DIN
- U6 pad 1: DISP_DATA -> DIN
Routing:
- net VCC: track 440.4 -> 28.2 mm, vias 21 -> 0
- net GND: track 351.7 -> 108.7 mm, vias 12 -> 19
- net DinMAX: track 0.00 -> 120.9 mm, vias 0 -> 1
- net DISP_DATA: track 70.9 -> 0.00 mm, vias 3 -> 0
- net CS1: track 57.9 -> 0.00 mm, vias 4 -> 0
- net Net-(U4-Pad22): track 0.00 -> 42.8 mm, vias 0 -> 1
- net Net-(U4-Pad15): track 0.00 -> 41.5 mm, vias 0 -> 1
- net Net-(D2-Pad2): track 41.5 -> 0.00 mm, vias 4 -> 0
- net Net-(U4-Pad17): track 0.00 -> 39.6 mm, vias 0 -> 1
- net Net-(D2-Pad12): track 36.6 -> 0.00 mm, vias 6 -> 0
- net CLK: track 36.0 -> 0.00 mm
- net Net-(U4-Pad21): track 0.00 -> 34.1 mm, vias 0 -> 1
- net Net-(D2-Pad11): track 0.00 -> 34.1 mm, vias 0 -> 1
- net Net-(BT1-Pad1): track 152.4 -> 119.6 mm, vias 7 -> 0
- net Net-(U4-Pad16): track 0.00 -> 32.6 mm, vias 0 -> 1
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